File: skna_project/ecg.kicad_sch (KiCad schematic)
At the start: 38 parts, among them J4 xRA_PAD, J5 xLA_PAD, U4 ADS1291RIPBS(TQFP)

Commit message: Replaced ADS129 with ADS8232
Parts:
- removed C13, C14: 4.7n, symbol Device:C_Small
- removed C14 (x2): 47p, symbol Device:C_Small
- removed C15: 10u, symbol Device:C_Small
- removed C16, C23, C25, C28, C31, C33: 0.1u, symbol Device:C_Small
- removed C21, C32, C34, C35: 2.2n, symbol Device:C_Small
- removed C22, C24, C27, C29, C30: 1u, symbol Device:C_Small
- removed C26: 1.5n, symbol Device:C_Small
- removed J4: xRA_PAD, symbol Connector:Screw_Terminal_01x01
- removed J5: xLA_PAD, symbol Connector:Screw_Terminal_01x01
- removed R14, R19, R20, R22, R23, R7, R8: 10M, symbol Device:R_Small
- removed R15, R16: 100k, symbol Device:R_Small
- removed R17: 1k, symbol Device:R_Small
- removed R18, R21: 39k, symbol Device:R_Small
- removed R22 (x2): 51k, symbol Device:R_Small
- removed U4: ADS1291RIPBS(TQFP), custom_components:ADS1291, symbol custom_regulator:ADS1291
Connections:
- no-connect marks 3 -> 0
